Commit message: Setting up sensors ...

File: softbot_description/urdf/astra.urdf.xacro (robot description, xacro)
@@ -28,5 +28,6 @@
       </collision>
       <inertial>
-        <mass value="0.564" />
+<!--        <mass value="0.564" />-->
+        <mass value="0.00564" />
         <origin xyz="0 0 0" />
         <inertia ixx="0.003881243" ixy="0.0" ixz="0.0"
@@ -65,5 +66,5 @@
           <sensor type="depth" name="camera">
               <always_on>true</always_on>
-              <update_rate>10.0</update_rate>
+              <update_rate>5.0</update_rate>
               <camera>
                   <horizontal_fov>${60.0*pi/180.0}</horizontal_fov>

File: softbot_description/urdf/ros_diff_drive.gazebo.xacro (robot description, xacro)
@@ -5,5 +5,6 @@
       <commandTopic>cmd_vel</commandTopic>
       <odometryTopic>odom</odometryTopic>
-      <odometryFrame>odom</odometryFrame>
+<!--      <odometryFrame>odom</odometryFrame>-->
+      <odometryFrame>world</odometryFrame>
       <odometrySource>world</odometrySource>
 <!--      <publishOdomTF>false</publishOdomTF>-->

File: softbot_description/urdf/softbot.urdf.xacro (robot description, xacro)
@@ -13,5 +13,5 @@
   <!-- Include other files-->
   <xacro:include filename="$(find softbot_description)/urdf/properties.xacro"/>
-  <xacro:include filename="$(find velodyne_description)/urdf/VLP-16.urdf.xacro"/>
+  <xacro:include filename="$(find softbot_description)/urdf/VLP-16.urdf.xacro"/>
   <xacro:include filename="$(find softbot_description)/urdf/astra.urdf.xacro" />
   <xacro:include filename="$(find softbot_description)/urdf/softbot.gazebo.macro.xacro"/>
@@ -35,5 +35,5 @@
       <origin xyz="-0.064 0 0.047" rpy="0 0 0"/>
       <geometry>
-<!--        <box size="0.266 0.266 0.094"/>-->
+        <!--        <box size="0.266 0.266 0.094"/>-->
         <box size="0.3 0.3 0.094"/>
       </geometry>
@@ -59,5 +59,5 @@
         <mesh filename="package://turtlebot3_description/meshes/wheels/left_tire.stl" scale="0.001 0.001 0.001"/>
       </geometry>
-      <material name="${color}"/>
+      <material name="black"/>
     </visual>
     <collision>
@@ -87,5 +87,5 @@
         <mesh filename="package://turtlebot3_description/meshes/wheels/right_tire.stl" scale="0.001 0.001 0.001"/>
       </geometry>
-      <material name="${color}"/>
+      <material name="black"/>
     </visual>
     <collision>
@@ -149,90 +149,105 @@
   </joint>
   <link name="imu_link"/>
-  <joint name="scan_joint" type="fixed">
-    <parent link="base_link"/>
-    <child link="base_scan"/>
-    <origin xyz="-0.064 0 0.122" rpy="0 0 0"/>
-  </joint>
-  <link name="base_scan">
-    <visual>
-      <origin xyz="0 0 0.0" rpy="0 0 0"/>
-      <geometry>
-        <mesh filename="package://turtlebot3_description/meshes/sensors/lds.stl" scale="0.001 0.001 0.001"/>
-      </geometry>
-      <material name="dark"/>
-    </visual>
-    <collision>
-      <origin xyz="0.015 0 -0.0065" rpy="0 0 0"/>
-      <geometry>
-        <cylinder length="0.0315" radius="0.055"/>
-      </geometry>
-    </collision>
-    <inertial>
-      <mass value="0.114" />
-      <origin xyz="0 0 0" />
-      <inertia ixx="0.001" ixy="0.0" ixz="0.0"
-               iyy="0.001" iyz="0.0"
-               izz="0.001" />
-    </inertial>
-  </link>
-  <joint name="camera_joint" type="fixed">
-    <origin xyz="0.073 -0.011 0.684" rpy="0 0.9 0"/>
-    <parent link="base_link"/>
-    <child link="camera_link"/>
-  </joint>
-  <link name="camera_link">
-<!--    <collision>-->
-<!--      <origin xyz="0.005 0.011 0.013" rpy="0 0 0"/>-->
-<!--      <geometry>-->
-<!--        <box size="0.015 0.030 0.027"/>-->
-<!--      </geometry>-->
-<!--    </collision>-->
-  </link>
-  <joint name="camera_rgb_joint" type="fixed">
-    <origin xyz="0.003 0.011 0.009" rpy="0 0 0"/>
-    <parent link="camera_link"/>
-    <child link="camera_rgb_frame"/>
-  </joint>
-  <link name="camera_rgb_frame"/>
-  <joint name="camera_rgb_optical_joint" type="fixed">
-    <origin xyz="0 0 0" rpy="-1.57 0 -1.57"/>
-    <parent link="camera_rgb_frame"/>
-    <child link="camera_rgb_optical_frame"/>
-  </joint>
-  <link name="camera_rgb_optical_frame"/>
-  <link name="lidar3d_support_link">
-    <visual>
-      <origin xyz="0 0 -0.1" rpy="0 0 0"/>
-<!--      <origin xyz="0 -0.1 -0.1" rpy="0 0 0"/>-->
-      <geometry>
-        <cylinder length="0.2" radius="0.004"/>
-<!--        <box size="0.1 0.3 0.094"/>-->
-      </geometry>
-        <material name="gray"/>
-    </visual>
-  </link>
-  <joint name="base_link_to_lidar3d_support_link" type="fixed">
-    <origin xyz="-.12 -.1 0.2" rpy="0 0 0"/>
-    <parent link="base_link"/>
-    <child link="lidar3d_support_link"/>
-  </joint>
-  <xacro:VLP-16 name="lidar3d" parent="lidar3d_support_link" topic="/lidar3d/points">
-    <origin xyz="0 0 0.001" rpy="0 0 0" />
+  <link name="platform_support_leg1_link">
+    <visual>
+      <origin xyz="0 0 -0.1" rpy="0 0 0"/>
+      <geometry>
+        <cylinder length="0.2" radius="0.004"/>
+      </geometry>
+      <material name="grey"/>
+    </visual>
+  </link>
+  <joint name="base_link_to_platform_support_leg1_link" type="fixed">
+    <parent link="base_link"/>
+    <child link="platform_support_leg1_link"/>
+    <origin xyz="-0.114 0.05 0.222" rpy="0 0 0"/>
+  </joint>
+  <link name="platform_support_leg2_link">
+    <visual>
+      <origin xyz="0 0 -0.1" rpy="0 0 0"/>
+      <geometry>
+        <cylinder length="0.2" radius="0.004"/>
+      </geometry>
+      <material name="grey"/>
+    </visual>
+  </link>
+  <joint name="base_link_to_platform_support_leg2_link" type="fixed">
+    <parent link="base_link"/>
+    <child link="platform_support_leg2_link"/>
+    <origin xyz="-0.114 -0.05 0.222" rpy="0 0 0"/>
+  </joint>
+  <link name="platform_support_leg3_link">
+    <visual>
+      <origin xyz="0 0 -0.1" rpy="0 0 0"/>
+      <geometry>
+        <cylinder length="0.2" radius="0.004"/>
+      </geometry>
+      <material name="grey"/>
+    </visual>
+  </link>
+  <joint name="base_link_to_platform_support_leg3_link" type="fixed">
+    <parent link="base_link"/>
+    <child link="platform_support_leg3_link"/>
+    <origin xyz="-0.014 0.05 0.222" rpy="0 0 0"/>
+  </joint>
+  <link name="platform_support_leg4_link">
+    <visual>
+      <origin xyz="0 0 -0.1" rpy="0 0 0"/>
+      <geometry>
+        <cylinder length="0.2" radius="0.004"/>
+      </geometry>
+      <material name="grey"/>
+    </visual>
+  </link>
+  <joint name="base_link_to_platform_support_leg4_link" type="fixed">
+    <parent link="base_link"/>
+    <child link="platform_support_leg4_link"/>
+    <origin xyz="-0.014 -0.05 0.222" rpy="0 0 0"/>
+  </joint>
+  <link name="lidar3d_plate_link">
+    <visual>
+      <origin xyz="0 0 0" rpy="0 0 0"/>
+      <geometry>
+        <box size="0.14 0.14 0.005"/>
+      </geometry>
+      <material name="grey"/>
+    </visual>
+  </link>
+  <joint name="platform_support_leg1_link_to_lidar3d_plate_link" type="fixed">
+    <parent link="platform_support_leg1_link"/>
+    <child link="lidar3d_plate_link"/>
+    <origin xyz="0.05 -0.05 0" rpy="0 0 0"/>
+  </joint>
+  <xacro:VLP-16 name="lidar3d" parent="lidar3d_plate_link" topic="/lidar3d/points">
+    <origin xyz="0 0 0" rpy="0 0 0" />
   </xacro:VLP-16>
-    <link name="front_camera_support_link">
-    <visual>
-      <origin xyz="0 0 -0.1" rpy="0 0 0"/>
-      <geometry>
-        <cylinder length="0.2" radius="0.004"/>
-      </geometry>
-        <material name="gray"/>
-    </visual>
-  </link>
-  <joint name="base_link_to_front_camera_support_link" type="fixed">
-    <origin xyz="-.12 .1 0.2" rpy="0 0 0"/>
-    <parent link="base_link"/>
-    <child link="front_camera_support_link"/>
-  </joint>
-  <xacro:sensor_astra prefix="front_camera" parent="front_camera_support_link">
+  <link name="front_left_camera_support_link">
+  </link>
+  <joint name="platform_support_leg3_link_to_front_left_camera_support_link" type="fixed">
+    <origin xyz="0.02 0 -0.09" rpy="0.01 -0.1 0.2"/>
+    <parent link="platform_support_leg3_link"/>
+    <child link="front_left_camera_support_link"/>
+  </joint>
+  <xacro:sensor_astra prefix="front_left_camera" parent="front_left_camera_support_link">
+    <origin xyz="0.02 0.07 0.015" rpy="0 0.0 0" />
+  </xacro:sensor_astra>
+  <link name="front_right_camera_support_link">
+  </link>
+  <joint name="platform_support_leg4_link_to_front_right_camera_support_link" type="fixed">
+    <origin xyz="0.02 0 -0.05" rpy="0.01 -0.05 -0.22"/>
+    <parent link="platform_support_leg4_link"/>
+    <child link="front_right_camera_support_link"/>
+  </joint>
+  <xacro:sensor_astra prefix="front_right_camera" parent="front_right_camera_support_link">
+    <origin xyz="0.02 0.07 0.015" rpy="0 0.0 0" />
+  </xacro:sensor_astra>
+  <link name="back_camera_support_link">
+  </link>
+  <joint name="platform_support_leg1_link_to_back_camera_support_link" type="fixed">
+    <origin xyz="-0.02 -0.05 -0.10" rpy="0.01 -0.15 3.14"/>
+    <parent link="platform_support_leg1_link"/>
+    <child link="back_camera_support_link"/>
+  </joint>
+  <xacro:sensor_astra prefix="back_camera" parent="back_camera_support_link">
     <origin xyz="0.02 0.07 0.015" rpy="0 0.0 0" />
   </xacro:sensor_astra>

Commit message: Removing dependencies from Eurico's iris_ur10e packages

File: softbot_description/urdf/astra.urdf.xacro (robot description, xacro)
@@ -17,5 +17,5 @@
         <origin xyz="-0.03 -0.06 0" rpy="${pi} 0 ${pi/2}"/>
         <geometry>
-          <mesh filename="package://ur_e_description/meshes/sensors/astra2.dae" scale="1 1 1"/>
+          <mesh filename="package://softbot_description/meshes/astra2/astra2.dae" scale="1 1 1"/>
         </geometry>
       </visual>
