Commit message: Setting rviz fixed frame to world_link

File: softbot_calibration/urdf/initial_estimate.urdf.xacro (robot description, xacro)
@@ -1,238 +1,30 @@
 <?xml version="1.0" ?>
-<robot name="softbot" version="1.0">
-  <material name="black">
-    <color rgba="0.0 0.0 0.0 1.0"/>
-  </material>
-  <material name="dark">
-    <color rgba="0.3 0.3 0.3 1.0"/>
-  </material>
-  <material name="light_black">
-    <color rgba="0.4 0.4 0.4 1.0"/>
-  </material>
-  <material name="blue">
-    <color rgba="0.0 0.0 0.8 1.0"/>
-  </material>
-  <material name="green">
-    <color rgba="0.0 0.8 0.0 1.0"/>
-  </material>
-  <material name="grey">
-    <color rgba="0.5 0.5 0.5 1.0"/>
-  </material>
-  <material name="orange">
-    <color rgba="1.0 0.4235294117647059 0.0392156862745098 1.0"/>
-  </material>
-  <material name="brown">
-    <color rgba="0.8705882352941177 0.8117647058823529 0.7647058823529411 1.0"/>
-  </material>
-  <material name="red">
-    <color rgba="0.8 0.0 0.0 1.0"/>
-  </material>
-  <material name="white">
-    <color rgba="1.0 1.0 1.0 1.0"/>
-  </material>
-  <material name="Yellow">
-    <color rgba="1.0 1.0 0.0 1.0"/>
-  </material>
-  <material name="Orange">
-    <color rgba="1.0 0.4 0.0 1.0"/>
-  </material>
-  <material name="Gray">
-    <color rgba="1.0 0.4 0.0 1.0"/>
-  </material>
-  <gazebo reference="base_link">
-    <material>Gazebo/Orange</material>
-  </gazebo>
-  <gazebo reference="base_link">
-    <sensor name="base_link" type="contact">
-      <update_rate>1000.0</update_rate>
-      <always_on>true</always_on>
-      <contact>
-        <collision>base_footprint_fixed_joint_lump__base_link_collision_collision</collision>
-      </contact>
-      <plugin filename="libgazebo_ros_bumper.so" name="base_link_contact_sensor_plugin">
-        <bumperTopicName>contact</bumperTopicName>
-        <frameName>world</frameName>
-      </plugin>
-    </sensor>
-  </gazebo>
-  <gazebo reference="wheel_left_link">
-    <mu1>0.1</mu1>
-    <mu2>0.1</mu2>
-    <kp>500000.0</kp>
-    <kd>10.0</kd>
-    <minDepth>0.001</minDepth>
-    <maxVel>0.1</maxVel>
-    <fdir1>1 0 0</fdir1>
-    <material>Gazebo/Orange</material>
-  </gazebo>
-  <gazebo reference="wheel_right_link">
-    <mu1>0.1</mu1>
-    <mu2>0.1</mu2>
-    <kp>500000.0</kp>
-    <kd>10.0</kd>
-    <minDepth>0.001</minDepth>
-    <maxVel>0.01</maxVel>
-    <fdir1>1 0 0</fdir1>
-    <material>Gazebo/Orange</material>
-  </gazebo>
-  <gazebo reference="caster_back_right_link">
-    <mu1>0.1</mu1>
-    <mu2>0.1</mu2>
-    <kp>1000000.0</kp>
-    <kd>100.0</kd>
-    <minDepth>0.001</minDepth>
-    <maxVel>1.0</maxVel>
-    <material>Gazebo/FlatBlack</material>
-  </gazebo>
-  <gazebo reference="caster_back_left_link">
-    <mu1>0.1</mu1>
-    <mu2>0.1</mu2>
-    <kp>1000000.0</kp>
-    <kd>100.0</kd>
-    <minDepth>0.001</minDepth>
-    <maxVel>1.0</maxVel>
-    <material>Gazebo/FlatBlack</material>
-  </gazebo>
-  <gazebo reference="imu_link">
-    <sensor name="imu" type="imu">
-      <always_on>true</always_on>
-      <visualize>True</visualize>
-    </sensor>
-    <material>Gazebo/Grey</material>
-  </gazebo>
-  <gazebo>
-    <plugin filename="libgazebo_ros_diff_drive.so" name="turtlebot3_waffle_pi_controller">
-      <commandTopic>cmd_vel</commandTopic>
-      <odometryTopic>odom</odometryTopic>
-      <odometryFrame>world</odometryFrame>
-      <odometrySource>world</odometrySource>
-      <publishOdomTF>true</publishOdomTF>
-      <robotBaseFrame>base_footprint</robotBaseFrame>
-      <publishWheelTF>false</publishWheelTF>
-      <publishTf>true</publishTf>
-      <publishWheelJointState>true</publishWheelJointState>
-      <legacyMode>false</legacyMode>
-      <updateRate>30</updateRate>
-      <leftJoint>wheel_left_joint</leftJoint>
-      <rightJoint>wheel_right_joint</rightJoint>
-      <wheelSeparation>0.287</wheelSeparation>
-      <wheelDiameter>0.066</wheelDiameter>
-      <wheelAcceleration>1</wheelAcceleration>
-      <wheelTorque>10</wheelTorque>
-      <rosDebugLevel>na</rosDebugLevel>
-    </plugin>
-  </gazebo>
-  <gazebo>
-    <plugin filename="libgazebo_ros_imu.so" name="imu_plugin">
-      <alwaysOn>true</alwaysOn>
-      <bodyName>imu_link</bodyName>
-      <frameName>imu_link</frameName>
-      <topicName>imu</topicName>
-      <serviceName>imu_service</serviceName>
-      <gaussianNoise>0.0</gaussianNoise>
-      <updateRate>200</updateRate>
-      <imu>
-        <noise>
-          <type>gaussian</type>
-          <rate>
-            <mean>0.0</mean>
-            <stddev>2e-4</stddev>
-            <bias_mean>0.0000075</bias_mean>
-            <bias_stddev>0.0000008</bias_stddev>
-          </rate>
-          <accel>
-            <mean>0.0</mean>
-            <stddev>1.7e-2</stddev>
-            <bias_mean>0.1</bias_mean>
-            <bias_stddev>0.001</bias_stddev>
-          </accel>
-        </noise>
-      </imu>
-    </plugin>
-  </gazebo>
-  <gazebo reference="base_scan">
-    <material>Gazebo/FlatBlack</material>
-    <sensor name="lds_lfcd_sensor" type="ray">
-      <pose>0 0 0 0 0 0</pose>
-      <visualize>False</visualize>
-      <update_rate>5</update_rate>
-      <ray>
-        <scan>
-          <horizontal>
-            <samples>360</samples>
-            <resolution>1</resolution>
-            <min_angle>0.0</min_angle>
-            <max_angle>6.28319</max_angle>
-          </horizontal>
-        </scan>
-        <range>
-          <min>0.120</min>
-          <max>3.5</max>
-          <resolution>0.015</resolution>
-        </range>
-        <noise>
-          <type>gaussian</type>
-          <mean>0.0</mean>
-          <stddev>0.01</stddev>
-        </noise>
-      </ray>
-      <plugin filename="libgazebo_ros_laser.so" name="gazebo_ros_lds_lfcd_controller">
-        <topicName>scan</topicName>
-        <frameName>base_scan</frameName>
-      </plugin>
-    </sensor>
-  </gazebo>
-  <gazebo reference="camera_rgb_frame">
-    <sensor name="Pi Camera" type="camera">
-      <always_on>true</always_on>
-      <visualize>False</visualize>
-      <camera>
-        <horizontal_fov>2.165595</horizontal_fov>
-        <image>
-          <width>1280</width>
-          <height>480</height>
-          <format>R8G8B8</format>
-        </image>
-        <clip>
-          <near>0.03</near>
-          <far>100</far>
-        </clip>
-      </camera>
-      <plugin filename="libgazebo_ros_camera.so" name="camera_controller">
-        <alwaysOn>true</alwaysOn>
-        <updateRate>30.0</updateRate>
-        <cameraName>camera</cameraName>
-        <frameName>camera_rgb_optical_frame</frameName>
-        <imageTopicName>rgb/image_raw</imageTopicName>
-        <cameraInfoTopicName>rgb/camera_info</cameraInfoTopicName>
-        <hackBaseline>0.07</hackBaseline>
-        <distortionK1>0.0</distortionK1>
-        <distortionK2>0.0</distortionK2>
-        <distortionK3>0.0</distortionK3>
-        <distortionT1>0.0</distortionT1>
-        <distortionT2>0.0</distortionT2>
-      </plugin>
-    </sensor>
-  </gazebo>
-  <gazebo reference="player_identifier_support_link">
-    <material>Gazebo/Grey</material>
-  </gazebo>
-  <gazebo reference="player_identifier_link">
-    <material>Gazebo/Orange</material>
-  </gazebo>
+<robot name="softbot" xmlns:xacro="http://ros.org/wiki/xacro">
+  <!--  Xacro description of turtlebot robot waffle pi used to play team hunt.-->
+  <!--  Miguel Riem Oliveira-->
+  <!--  PARI, November 2020-->
+  <!--Args are local, properties are global, so we copy the values of the arguments to the properties-->
+  <xacro:arg name="name" default="softbot" />
+  <xacro:arg name="color" default="Orange" /> <!-- e.g. Red, Orange. Must exist in Gazebo/Colors and be defined in properties.xacro.-->
+  <!--Properties are global so they can be viewed from inside the included xacros-->
+  <!--  args are used with $(arg arg_name), properties are used as ${property_name}-->
+  <xacro:property name="name" value="$(arg name)"/>
+  <xacro:property name="color" value="$(arg color)"/>
+  <!-- Include other files-->
+  <xacro:include filename="$(find softbot_description)/urdf/properties.xacro"/>
+  <xacro:include filename="$(find softbot_description)/urdf/VLP-16.urdf.xacro"/>
+  <xacro:include filename="$(find softbot_description)/urdf/astra.urdf.xacro" />
+  <xacro:include filename="$(find softbot_description)/urdf/softbot.gazebo.macro.xacro"/>
+  <xacro:gazebo_macro color="$(arg color)" laser_visual="false" camera_visual="false" imu_visual="true"/>
+  <!-- Links and joints-->
   <link name="base_footprint"/>
   <joint name="base_joint" type="fixed">
-    <origin xyz="0.0 0.0 0.01" rpy="0.0 0.0 0.0"/>
     <parent link="base_footprint"/>
-    <child link="base_link"/>
+    <child link="base_link" />
+    <origin xyz="0 0 0.010" rpy="0 0 0"/>
   </joint>
   <link name="base_link">
-    <inertial>
-      <origin xyz="0.0 0.0 0.0" rpy="0.0 0.0 0.0"/>
-      <mass value="1.3729096"/>
-      <inertia ixx="0.0087002718" ixy="-4.7576583e-05" ixz="0.00011160499" iyy="0.0086195418" iyz="-3.5422299e-06" izz="0.014612727"/>
-    </inertial>
-    <visual>
-      <origin xyz="-0.064 0.0 0.0" rpy="0.0 0.0 0.0"/>
+    <visual>
+      <origin xyz="-0.064 0 0.0" rpy="0 0 0"/>
       <geometry>
         <mesh filename="package://turtlebot3_description/meshes/bases/waffle_pi_base.stl" scale="0.001 0.001 0.001"/>
@@ -240,25 +32,28 @@
       <material name="light_black"/>
     </visual>
-    <collision>
-      <origin xyz="-0.064 0.0 0.047" rpy="0.0 0.0 0.0"/>
-      <geometry>
+    <collision name="base_link_collision">
+      <origin xyz="-0.064 0 0.047" rpy="0 0 0"/>
+      <geometry>
+        <!--        <box size="0.266 0.266 0.094"/>-->
         <box size="0.3 0.3 0.094"/>
       </geometry>
     </collision>
+    <inertial>
+      <origin xyz="0 0 0" rpy="0 0 0"/>
+      <mass value="1.3729096e+00"/>
+      <inertia ixx="8.7002718e-03" ixy="-4.7576583e-05" ixz="1.1160499e-04"
+               iyy="8.6195418e-03" iyz="-3.5422299e-06"
+               izz="1.4612727e-02" />
+    </inertial>
   </link>
   <joint name="wheel_left_joint" type="continuous">
-    <origin xyz="0.0 0.144 0.023" rpy="-1.57 0.0 0.0"/>
-    <axis xyz="0.0 0.0 1.0"/>
     <parent link="base_link"/>
     <child link="wheel_left_link"/>
+    <origin xyz="0.0 0.144 0.023" rpy="-1.57 0 0"/>
+    <axis xyz="0 0 1"/>
   </joint>
   <link name="wheel_left_link">
-    <inertial>
-      <origin xyz="0.0 0.0 0.0" rpy="0 0 0"/>
-      <mass value="0.02849894"/>
-      <inertia ixx="1.117558e-05" ixy="-4.2369783e-11" ixz="-5.9381719e-09" iyy="1.1192413e-05" iyz="-1.4400107e-11" izz="2.0712558e-05"/>
-    </inertial>
-    <visual>
-      <origin xyz="0.0 0.0 0.0" rpy="1.57 0.0 0.0"/>
+    <visual>
+      <origin xyz="0 0 0" rpy="1.57 0 0"/>
       <geometry>
         <mesh filename="package://turtlebot3_description/meshes/wheels/left_tire.stl" scale="0.001 0.001 0.001"/>
@@ -267,24 +62,26 @@
     </visual>
     <collision>
-      <origin xyz="0.0 0.0 0.0" rpy="0.0 0.0 0.0"/>
-      <geometry>
-        <cylinder radius="0.033" length="0.018"/>
-      </geometry>
-    </collision>
+      <origin xyz="0 0 0" rpy="0 0 0"/>
+      <geometry>
+        <cylinder length="0.018" radius="0.033"/>
+      </geometry>
+    </collision>
+    <inertial>
+      <origin xyz="0 0 0" />
+      <mass value="2.8498940e-02" />
+      <inertia ixx="1.1175580e-05" ixy="-4.2369783e-11" ixz="-5.9381719e-09"
+               iyy="1.1192413e-05" iyz="-1.4400107e-11"
+               izz="2.0712558e-05" />
+    </inertial>
   </link>
   <joint name="wheel_right_joint" type="continuous">
-    <origin xyz="0.0 -0.144 0.023" rpy="-1.57 0.0 0.0"/>
-    <axis xyz="0.0 0.0 1.0"/>
     <parent link="base_link"/>
     <child link="wheel_right_link"/>
+    <origin xyz="0.0 -0.144 0.023" rpy="-1.57 0 0"/>
+    <axis xyz="0 0 1"/>
   </joint>
   <link name="wheel_right_link">
-    <inertial>
-      <origin xyz="0.0 0.0 0.0" rpy="0 0 0"/>
-      <mass value="0.02849894"/>
-      <inertia ixx="1.117558e-05" ixy="-4.2369783e-11" ixz="-5.9381719e-09" iyy="1.1192413e-05" iyz="-1.4400107e-11" izz="2.0712558e-05"/>
-    </inertial>
-    <visual>
-      <origin xyz="0.0 0.0 0.0" rpy="1.57 0.0 0.0"/>
+    <visual>
+      <origin xyz="0 0 0" rpy="1.57 0 0"/>
       <geometry>
         <mesh filename="package://turtlebot3_description/meshes/wheels/right_tire.stl" scale="0.001 0.001 0.001"/>
@@ -293,57 +90,68 @@
     </visual>
     <collision>
-      <origin xyz="0.0 0.0 0.0" rpy="0.0 0.0 0.0"/>
-      <geometry>
-        <cylinder radius="0.033" length="0.018"/>
-      </geometry>
-    </collision>
+      <origin xyz="0 0 0" rpy="0 0 0"/>
+      <geometry>
+        <cylinder length="0.018" radius="0.033"/>
+      </geometry>
+    </collision>
+    <inertial>
+      <origin xyz="0 0 0" />
+      <mass value="2.8498940e-02" />
+      <inertia ixx="1.1175580e-05" ixy="-4.2369783e-11" ixz="-5.9381719e-09"
+               iyy="1.1192413e-05" iyz="-1.4400107e-11"
+               izz="2.0712558e-05" />
+    </inertial>
   </link>
   <joint name="caster_back_right_joint" type="fixed">
-    <origin xyz="-0.177 -0.064 -0.004" rpy="-1.57 0.0 0.0"/>
     <parent link="base_link"/>
     <child link="caster_back_right_link"/>
+    <origin xyz="-0.177 -0.064 -0.004" rpy="-1.57 0 0"/>
   </joint>
   <link name="caster_back_right_link">
-    <inertial>
-      <origin xyz="0.0 0.0 0.0" rpy="0 0 0"/>
-      <mass value="0.005"/>
-      <inertia ixx="0.001" ixy="0.0" ixz="0.0" iyy="0.001" iyz="0.0" izz="0.001"/>
-    </inertial>
-    <collision>
-      <origin xyz="0.0 0.001 0.0" rpy="0.0 0.0 0.0"/>
-      <geometry>
-        <box size="0.03 0.009 0.02"/>
-      </geometry>
-    </collision>
+    <collision>
+      <origin xyz="0 0.001 0" rpy="0 0 0"/>
+      <geometry>
+        <box size="0.030 0.009 0.020"/>
+      </geometry>
+    </collision>
+    <inertial>
+      <origin xyz="0 0 0" />
+      <mass value="0.005" />
+      <inertia ixx="0.001" ixy="0.0" ixz="0.0"
+               iyy="0.001" iyz="0.0"
+               izz="0.001" />
+    </inertial>
   </link>
   <joint name="caster_back_left_joint" type="fixed">
-    <origin xyz="-0.177 0.064 -0.004" rpy="-1.57 0.0 0.0"/>
     <parent link="base_link"/>
     <child link="caster_back_left_link"/>
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
File: softbot_description/urdf/VLP-16.urdf.xacro (robot description, xacro)
@@ -2,5 +2,5 @@
 <robot xmlns:xacro="http://www.ros.org/wiki/xacro" name="VLP-16">
   <xacro:property name="M_PI" value="3.1415926535897931" />
-  <xacro:macro name="VLP-16" params="*origin parent:=base_link name:=velodyne topic:=/velodyne_points organize_cloud:=false hz:=5 lasers:=16 samples:=1875 collision_range:=0.3 min_range:=0.9 max_range:=130.0 noise:=0.008 min_angle:=-${M_PI} max_angle:=${M_PI} gpu:=false">
+  <xacro:macro name="VLP-16" params="*origin parent:=base_link name:=velodyne topic:=/velodyne_points organize_cloud:=false hz:=10 lasers:=16 samples:=1875 collision_range:=0.3 min_range:=0.9 max_range:=130.0 noise:=0.008 min_angle:=-${M_PI} max_angle:=${M_PI} gpu:=false">
     <joint name="${name}_base_mount_joint" type="fixed">
       <xacro:insert_block name="origin" />

File: softbot_description/urdf/astra.urdf.xacro (robot description, xacro)
@@ -66,5 +66,5 @@
           <sensor type="depth" name="camera">
               <always_on>true</always_on>
-              <update_rate>5.0</update_rate>
+              <update_rate>10.0</update_rate>
               <camera>
                   <horizontal_fov>${60.0*pi/180.0}</horizontal_fov>

File: softbot_description/urdf/softbot.gazebo.macro.xacro (robot description, xacro)
@@ -132,47 +132,4 @@
     </sensor>
   </gazebo>
-  <!--link : https://www.raspberrypi.org/documentation/hardware/camera/-->
-  <gazebo reference="camera_rgb_frame">
-    <sensor type="camera" name="Pi Camera">
-      <always_on>true</always_on>
-      <visualize>${camera_visual}</visualize>
-      <camera>
-<!--        <horizontal_fov>1.085595</horizontal_fov>-->
-        <horizontal_fov>2.165595</horizontal_fov>
-        <image>
-<!--          <width>640</width>-->
-          <width>1280</width>
-<!--          <width>640</width>-->
-<!--          <height>480</height>-->
-          <height>480</height>
-          <format>R8G8B8</format>
-        </image>
-        <clip>
-          <near>0.03</near>
-          <far>100</far>
-        </clip>
-      </camera>
-      <plugin name="camera_controller" filename="libgazebo_ros_camera.so">
-        <alwaysOn>true</alwaysOn>
-        <updateRate>30.0</updateRate>
-        <cameraName>camera</cameraName>
-        <frameName>camera_rgb_optical_frame</frameName>
-        <imageTopicName>rgb/image_raw</imageTopicName>
-        <cameraInfoTopicName>rgb/camera_info</cameraInfoTopicName>
-        <hackBaseline>0.07</hackBaseline>
-        <distortionK1>0.0</distortionK1>
-        <distortionK2>0.0</distortionK2>
-        <distortionK3>0.0</distortionK3>
-        <distortionT1>0.0</distortionT1>
-        <distortionT2>0.0</distortionT2>
-      </plugin>
-    </sensor>
-  </gazebo>
-  <gazebo reference="player_identifier_support_link">
-    <material>Gazebo/Grey</material>
-  </gazebo>
-  <gazebo reference="player_identifier_link">
-    <material>Gazebo/${color}</material>
-  </gazebo>
 </xacro:macro>
 </robot>

File: softbot_description/urdf/softbot.urdf.xacro (robot description, xacro)
@@ -225,5 +225,5 @@
   </link>
   <joint name="platform_support_leg3_link_to_front_left_camera_support_link" type="fixed">
-    <origin xyz="0.02 0 -0.09" rpy="0.01 -0.1 0.2"/>
+    <origin xyz="0.02 0 -0.09" rpy="0.01 -0.35 0.2"/>
     <parent link="platform_support_leg3_link"/>
     <child link="front_left_camera_support_link"/>
@@ -235,5 +235,5 @@
   </link>
   <joint name="platform_support_leg4_link_to_front_right_camera_support_link" type="fixed">
-    <origin xyz="0.02 0 -0.05" rpy="0.01 -0.05 -0.22"/>
+    <origin xyz="0.02 0 -0.05" rpy="0.01 -0.35 -0.22"/>
     <parent link="platform_support_leg4_link"/>
     <child link="front_right_camera_support_link"/>
@@ -245,5 +245,5 @@
   </link>
   <joint name="platform_support_leg1_link_to_back_camera_support_link" type="fixed">
-    <origin xyz="-0.02 -0.05 -0.10" rpy="0.01 -0.15 3.14"/>
+    <origin xyz="-0.02 -0.05 -0.10" rpy="0.01 -0.35 3.14"/>
     <parent link="platform_support_leg1_link"/>
     <child link="back_camera_support_link"/>

Commit message: new dataset3

File: softbot_calibration/urdf/initial_estimate.urdf.xacro (robot description, xacro)
@@ -242,13 +242,13 @@
     <origin xyz="0.02 0.07 0.015" rpy="0 0.0 0" />
   </xacro:sensor_astra>
-  <link name="back_camera_support_link">
-  </link>
-  <joint name="platform_support_leg1_link_to_back_camera_support_link" type="fixed">
-    <origin xyz="-0.02 -0.05 -0.10" rpy="0.01 -0.35 3.14"/>
-    <parent link="platform_support_leg1_link"/>
-    <child link="back_camera_support_link"/>
-  </joint>
-  <xacro:sensor_astra prefix="back_camera" parent="back_camera_support_link">
-    <origin xyz="0.02 0.07 0.015" rpy="0 0.0 0" />
-  </xacro:sensor_astra>
+<!--  <link name="back_camera_support_link">-->
+<!--  </link>-->
+<!--  <joint name="platform_support_leg1_link_to_back_camera_support_link" type="fixed">-->
+<!--    <origin xyz="-0.02 -0.05 -0.10" rpy="0.01 -0.35 3.14"/>-->
+<!--    <parent link="platform_support_leg1_link"/>-->
+<!--    <child link="back_camera_support_link"/>-->
+<!--  </joint>-->
+<!--  <xacro:sensor_astra prefix="back_camera" parent="back_camera_support_link">-->
+<!--    <origin xyz="0.02 0.07 0.015" rpy="0 0.0 0" />-->
+<!--  </xacro:sensor_astra>-->
 </robot>
