Commit message: Setting up calibration of softbot.

File: softbot_calibration/urdf/optimized_w_pattern.urdf.xacro (robot description, xacro)
@@ -646,3 +646,17 @@
     </sensor>
   </gazebo>
+  <link name="pattern_link">
+    <origin xyz="0 0 0" rpy="0 0 0"/>
+    <visual name="pattern_1_visual">
+      <origin xyz="0 0 0" rpy="0 0 0"/>
+      <geometry>
+        <mesh filename="package://atom_worlds/pattern/models/charuco_800x600_5x5_100/charuco_800x600_5x5_100.dae"/>
+      </geometry>
+    </visual>
+  </link>
+  <joint name="world-pattern_link" type="fixed">
+    <origin xyz="2.1279017804298648 0.29816703408043743 0.7927179887872843" rpy="-1.7842967447208273 -0.47461976188783866 -1.184754775705039"/>
+    <parent link="world"/>
+    <child link="pattern_link"/>
+  </joint>
 </robot>

Commit message: deleting old files and fixing itneractive pattern

File: softbot_calibration/urdf/optimized_w_pattern.urdf.xacro (robot description, xacro)
@@ -646,3 +646,17 @@
     </sensor>
   </gazebo>
+  <link name="pattern_link">
+    <origin xyz="0 0 0" rpy="0 0 0"/>
+    <visual name="pattern_1_visual">
+      <origin xyz="0 0 0" rpy="0 0 0"/>
+      <geometry>
+        <mesh filename="package://atom_worlds/pattern/models/charuco_800x600_5x5_100/charuco_800x600_5x5_100.dae"/>
+      </geometry>
+    </visual>
+  </link>
+  <joint name="world-pattern_link" type="fixed">
+    <origin xyz="1.2738060711451347 0.5273504656342143 0.9196604366186216" rpy="-1.5738202028369945 -0.7454204558294389 -1.6041199074449553"/>
+    <parent link="world"/>
+    <child link="pattern_link"/>
+  </joint>
 </robot>
