Commit message: changes on README

File: softbot_calibration/urdf/optimized.urdf.xacro (robot description, xacro)
@@ -374,5 +374,5 @@
   </joint>
   <joint name="lidar3d_base_mount_joint" type="fixed">
-    <origin xyz="1.5424578888797933e-16 -4.404261471365649e-16 -4.4408905585090867e-16" rpy="-1.7490387609158247e-16 4.4376732045088474e-16 -4.440851232392048e-16"/>
+    <origin xyz="4.438044141947997e-16 -3.3567055786269235e-16 -4.440891593897578e-16" rpy="-4.4408913177390826e-16 4.4401323532796685e-16 -4.440890130132144e-16"/>
     <parent link="lidar3d_plate_link"/>
     <child link="lidar3d_base_link"/>
@@ -467,5 +467,5 @@
   </joint>
   <joint name="front_left_camera_joint" type="fixed">
-    <origin xyz="0.016993239853372286 0.08232906859814623 0.012309034931527756" rpy="-0.000899532039260679 0.000833432616274603 0.0006886817182980605"/>
+    <origin xyz="0.019128951150184714 0.09622477198272436 0.011491975429385355" rpy="-0.00011102593929324018 0.000432866349022773 -0.0008815743252232054"/>
     <parent link="front_left_camera_support_link"/>
     <child link="front_left_camera_link"/>
@@ -560,5 +560,5 @@
   </joint>
   <joint name="front_right_camera_joint" type="fixed">
-    <origin xyz="0.022424827608530633 0.0828675417079197 0.011706747566180247" rpy="-0.0010272847974285024 0.0008349250695681769 0.0006289634030883567"/>
+    <origin xyz="0.018678763660725434 0.09589135336666572 0.011603158264384503" rpy="-0.0001820055780953038 0.00042645457637731257 -0.0007605714467599055"/>
     <parent link="front_right_camera_support_link"/>
     <child link="front_right_camera_link"/>

Commit message: added ipg gif and tables

File: softbot_calibration/urdf/optimized.urdf.xacro (robot description, xacro)
@@ -374,5 +374,5 @@
   </joint>
   <joint name="lidar3d_base_mount_joint" type="fixed">
-    <origin xyz="0.00028433405212385934 -5.248709756694661e-05 -0.00036969732491750777" rpy="-0.001337135226344172 0.0007385061159705848 -0.01340818571269933"/>
+    <origin xyz="-0.0023070810875422706 0.0024361113444771954 0.004090923931357919" rpy="0.006279112325167193 0.002809371202464486 -0.009565623283655667"/>
     <parent link="lidar3d_plate_link"/>
     <child link="lidar3d_base_link"/>
@@ -494,5 +494,5 @@
   </gazebo>
   <joint name="front_left_camera_rgb_joint" type="fixed">
-    <origin xyz="4.4315840342871636e-16 -0.04499999999999956 -1.1816846761836635e-16" rpy="7.75134384209754e-17 -2.4776014121687433e-16 4.4408920582567643e-16"/>
+    <origin xyz="7.084724016297851e-17 -0.04499999999999956 7.319932922969775e-17" rpy="-3.6538387428591485e-16 4.221148759943811e-16 4.4372629863365957e-16"/>
     <parent link="front_left_camera_link"/>
     <child link="front_left_camera_rgb_frame"/>
@@ -587,5 +587,5 @@
   </gazebo>
   <joint name="front_right_camera_rgb_joint" type="fixed">
-    <origin xyz="0.008295367367715047 -0.04164269242089581 -0.0015686258745966507" rpy="-0.0025047352023531344 0.000296850902231802 -0.0010525278953417798"/>
+    <origin xyz="0.002396265437130516 -0.04157874977702832 -0.003021812333265874" rpy="-0.0057467864963438335 -0.0010398140950835305 -0.002400262309175431"/>
     <parent link="front_right_camera_link"/>
     <child link="front_right_camera_rgb_frame"/>

File: softbot_calibration/urdf/optimized_w_pattern.urdf.xacro (robot description, xacro)
@@ -374,5 +374,5 @@
   </joint>
   <joint name="lidar3d_base_mount_joint" type="fixed">
-    <origin xyz="0.00028433405212385934 -5.248709756694661e-05 -0.00036969732491750777" rpy="-0.001337135226344172 0.0007385061159705848 -0.01340818571269933"/>
+    <origin xyz="-0.0023070810875422706 0.0024361113444771954 0.004090923931357919" rpy="0.006279112325167193 0.002809371202464486 -0.009565623283655667"/>
     <parent link="lidar3d_plate_link"/>
     <child link="lidar3d_base_link"/>
@@ -494,5 +494,5 @@
   </gazebo>
   <joint name="front_left_camera_rgb_joint" type="fixed">
-    <origin xyz="4.4315840342871636e-16 -0.04499999999999956 -1.1816846761836635e-16" rpy="7.75134384209754e-17 -2.4776014121687433e-16 4.4408920582567643e-16"/>
+    <origin xyz="7.084724016297851e-17 -0.04499999999999956 7.319932922969775e-17" rpy="-3.6538387428591485e-16 4.221148759943811e-16 4.4372629863365957e-16"/>
     <parent link="front_left_camera_link"/>
     <child link="front_left_camera_rgb_frame"/>
@@ -587,5 +587,5 @@
   </gazebo>
   <joint name="front_right_camera_rgb_joint" type="fixed">
-    <origin xyz="0.008295367367715047 -0.04164269242089581 -0.0015686258745966507" rpy="-0.0025047352023531344 0.000296850902231802 -0.0010525278953417798"/>
+    <origin xyz="0.002396265437130516 -0.04157874977702832 -0.003021812333265874" rpy="-0.0057467864963438335 -0.0010398140950835305 -0.002400262309175431"/>
     <parent link="front_right_camera_link"/>
     <child link="front_right_camera_rgb_frame"/>
@@ -656,5 +656,5 @@
   </link>
   <joint name="world-pattern_link" type="fixed">
-    <origin xyz="1.2738060711451347 0.5273504656342143 0.9196604366186216" rpy="-1.5738202028369945 -0.7454204558294389 -1.6041199074449553"/>
+    <origin xyz="1.268258447034737 0.5274889285614608 0.9159035598706413" rpy="-1.5707817211334032 -0.7490378691961472 -1.6017391965079912"/>
     <parent link="world"/>
     <child link="pattern_link"/>

Commit message: adding docs

File: softbot_calibration/urdf/optimized.urdf.xacro (robot description, xacro)
@@ -374,5 +374,5 @@
   </joint>
   <joint name="lidar3d_base_mount_joint" type="fixed">
-    <origin xyz="-0.0023070810875422706 0.0024361113444771954 0.004090923931357919" rpy="0.006279112325167193 0.002809371202464486 -0.009565623283655667"/>
+    <origin xyz="-0.0015142375046177249 -0.0022052142273190152 -0.000283564068925264" rpy="-0.007757658250765604 0.0009838709879697281 -0.014847674947914611"/>
     <parent link="lidar3d_plate_link"/>
     <child link="lidar3d_base_link"/>
@@ -494,5 +494,5 @@
   </gazebo>
   <joint name="front_left_camera_rgb_joint" type="fixed">
-    <origin xyz="7.084724016297851e-17 -0.04499999999999956 7.319932922969775e-17" rpy="-3.6538387428591485e-16 4.221148759943811e-16 4.4372629863365957e-16"/>
+    <origin xyz="-4.399872653456163e-16 -0.04499999999999956 3.1045954087761856e-16" rpy="-4.440829884921592e-16 4.4301780635402403e-16 4.438903032319087e-16"/>
     <parent link="front_left_camera_link"/>
     <child link="front_left_camera_rgb_frame"/>
@@ -587,5 +587,5 @@
   </gazebo>
   <joint name="front_right_camera_rgb_joint" type="fixed">
-    <origin xyz="0.002396265437130516 -0.04157874977702832 -0.003021812333265874" rpy="-0.0057467864963438335 -0.0010398140950835305 -0.002400262309175431"/>
+    <origin xyz="0.002030911322794242 -0.03938584552044518 -1.2175099096372358e-05" rpy="-0.005222638857532736 0.001007139992505166 -0.0037596367537089353"/>
     <parent link="front_right_camera_link"/>
     <child link="front_right_camera_rgb_frame"/>

File: softbot_calibration/urdf/optimized_w_pattern.urdf.xacro (robot description, xacro)
@@ -374,5 +374,5 @@
   </joint>
   <joint name="lidar3d_base_mount_joint" type="fixed">
-    <origin xyz="-0.0023070810875422706 0.0024361113444771954 0.004090923931357919" rpy="0.006279112325167193 0.002809371202464486 -0.009565623283655667"/>
+    <origin xyz="-0.0015142375046177249 -0.0022052142273190152 -0.000283564068925264" rpy="-0.007757658250765604 0.0009838709879697281 -0.014847674947914611"/>
     <parent link="lidar3d_plate_link"/>
     <child link="lidar3d_base_link"/>
@@ -494,5 +494,5 @@
   </gazebo>
   <joint name="front_left_camera_rgb_joint" type="fixed">
-    <origin xyz="7.084724016297851e-17 -0.04499999999999956 7.319932922969775e-17" rpy="-3.6538387428591485e-16 4.221148759943811e-16 4.4372629863365957e-16"/>
+    <origin xyz="-4.399872653456163e-16 -0.04499999999999956 3.1045954087761856e-16" rpy="-4.440829884921592e-16 4.4301780635402403e-16 4.438903032319087e-16"/>
     <parent link="front_left_camera_link"/>
     <child link="front_left_camera_rgb_frame"/>
@@ -587,5 +587,5 @@
   </gazebo>
   <joint name="front_right_camera_rgb_joint" type="fixed">
-    <origin xyz="0.002396265437130516 -0.04157874977702832 -0.003021812333265874" rpy="-0.0057467864963438335 -0.0010398140950835305 -0.002400262309175431"/>
+    <origin xyz="0.002030911322794242 -0.03938584552044518 -1.2175099096372358e-05" rpy="-0.005222638857532736 0.001007139992505166 -0.0037596367537089353"/>
     <parent link="front_right_camera_link"/>
     <child link="front_right_camera_rgb_frame"/>
@@ -656,5 +656,5 @@
   </link>
   <joint name="world-pattern_link" type="fixed">
-    <origin xyz="1.268258447034737 0.5274889285614608 0.9159035598706413" rpy="-1.5707817211334032 -0.7490378691961472 -1.6017391965079912"/>
+    <origin xyz="1.273180549764564 0.5275071795462576 0.9180241714021727" rpy="-1.57238029953394 -0.7458089302748174 -1.6092354412755343"/>
     <parent link="world"/>
     <child link="pattern_link"/>
